File: SchrackPanel/PCB/MECHANICAL.kicad_sch (KiCad schematic)
At the start: 14 parts, among them J1 RJ45, J2 RJ45, J3 RJ45, J4 RJ45, J5 RJ45, J6 RJ45, J7 RJ45, J8 RJ45

Commit message: 3d updates
inductors, tacticle buttons
Parts:
- J1, J2, J3, J4, J5, J6, J7, J8: footprint Connector_RJ:RJ45_Amphenol_54602-x08_Horizontal -> Schrack_brd:RJ45_Amphenol_54602-x08_Horizontal
Changed lines of the file:
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@@
 			)
 		)
-		(property "Footprint" "Connector_RJ:RJ45_Amphenol_54602-x08_Horizontal"
+		(property "Footprint" "Schrack_brd:RJ45_Amphenol_54602-x08_Horizontal"
 			(at 66.675 48.26 90)
 			(effects
@@
 			)
 		)
-		(property "Footprint" "Connector_RJ:RJ45_Amphenol_54602-x08_Horizontal"
+		(property "Footprint" "Schrack_brd:RJ45_Amphenol_54602-x08_Horizontal"
 			(at 259.715 48.26 90)
 			(effects
@@
 			)
 		)
-		(property "Footprint" "Connector_RJ:RJ45_Amphenol_54602-x08_Horizontal"
+		(property "Footprint" "Schrack_brd:RJ45_Amphenol_54602-x08_Horizontal"
 			(at 225.425 48.26 90)
 			(effects
@@
 			)
 		)
-		(property "Footprint" "Connector_RJ:RJ45_Amphenol_54602-x08_Horizontal"
+		(property "Footprint" "Schrack_brd:RJ45_Amphenol_54602-x08_Horizontal"
 			(at 98.425 48.26 90)
 			(effects
@@
 			)
 		)
-		(property "Footprint" "Connector_RJ:RJ45_Amphenol_54602-x08_Horizontal"
+		(property "Footprint" "Schrack_brd:RJ45_Amphenol_54602-x08_Horizontal"
 			(at 33.655 48.26 90)
 			(effects
@@
 			)
 		)
-		(property "Footprint" "Connector_RJ:RJ45_Amphenol_54602-x08_Horizontal"
+		(property "Footprint" "Schrack_brd:RJ45_Amphenol_54602-x08_Horizontal"
 			(at 193.675 48.26 90)
 			(effects
@@
 			)
 		)
-		(property "Footprint" "Connector_RJ:RJ45_Amphenol_54602-x08_Horizontal"
+		(property "Footprint" "Schrack_brd:RJ45_Amphenol_54602-x08_Horizontal"
 			(at 130.175 48.26 90)
 			(effects
@@
 			)
 		)
-		(property "Footprint" "Connector_RJ:RJ45_Amphenol_54602-x08_Horizontal"
+		(property "Footprint" "Schrack_brd:RJ45_Amphenol_54602-x08_Horizontal"
 			(at 161.925 48.26 90)
 			(effects
