File: SchrackCounter/PCB/SchrackCounterPrototype/LOGIC_CONTROL.kicad_sch (KiCad schematic)
At the start: 15 parts, among them J1 Conn_01x05_Pin, SW1 SW_Push, SW2 SW_Push, SW3 SW_Push

Commit message: schrack multiclock schematic update
Just regular updates
Parts:
- added BZ1: Buzzer, Buzzer_Beeper:Buzzer_15x7.5RM7.6, symbol Device:Buzzer
- added R8: 0R, Resistor_THT:R_Axial_DIN0207_L6.3mm_D2.5mm_P10.16mm_Horizontal, symbol Device:R
Connections:
- net GND: now also BZ1.2 (-)
- new net: BZ1.1 (+), R8.2
- new net BZ1_PWM: R8.1
