File: SchrackMulticlock/PCB/SchrackMulticlock/SchrackMulticlock.kicad_pcb (KiCad board)
At the start: 4 copper layers, 98.5 x 88.5 mm, 65 parts, among them J1 TYPE-C-31-M-12 (USB C CONN), J2 MEM2067-02-180-00-A_REVB, SW1 SW_SPST, SW2 SW_Push, SW3 SW_Push, SW4 SW_Push, SW5 SW_Push, SW6 SW_Push, U1 LM1084-3.3, U2 LDD080AUE-101A, U3 LTD080AUE-103A, U4 LDD080AUE-101A, U5 MAX7219, U6 ESP32-S3-WROOM-2, U7 USBLC6-2SC6

Commit message: SchrackMulticlock and Counter update
Schematic update for both
PCB update for Counter
Parts:
- BT1: footprint Schrack_brd:SOLDER_PADS -> Battery:BatteryHolder_TruPower_BH-331P_3xAA
- C1, C10, C11, C13, C15, C16, C2, C3, C4, C5, C6, C7, C8, R1, R10, R11, R12, R13, R15, R16, R2, R3, R4, R5, R6, R7, U1, U5, U7: moved to F.Cu
- C12: value 100nF.en -> 100nF; moved to F.Cu
- C14: value 100nF.boot -> 100nF; moved to F.Cu
- D4: footprint LED_SMD:LED_0805_2012Metric_Pad1.15x1.40mm_HandSolder -> LED_SMD:LED_Cree-PLCC4_3.2x2.8mm_CCW
- R14: value 10k.mcu -> 10k; moved to F.Cu
- U3: value LTD080AUE-103A -> LDD080AUE-101A; footprint Schrack_brd:WENRUN_LTD080x_7segment_3dig -> Schrack_brd:WENRUN_LDD080x_7segment_2dig
- moved D_EXT3 231.1 mm to (4.20, 124.5), turned to 0 degrees
- moved D_EXT2 222.2 mm to (4.20, 116.7), turned to 0 degrees
- moved D7 216.8 mm to (28.2, 137.8)
- moved D_EXT1 213.7 mm to (4.20, 108.9), turned to 0 degrees
- moved D6 213.5 mm to (28.2, 134.8)
- moved D5 211.7 mm to (28.2, 131.7)
- moved R4 208.4 mm to (27.1, 112.9), turned to 0 degrees
- moved C9 206.8 mm to (3.13, 135.0), turned to 0 degrees
- moved R10 204.7 mm to (31.9, 112.9), turned to 0 degrees
- moved D4 203.8 mm to (38.8, 132.1)
- moved R11 203.1 mm to (31.9, 115.9), turned to 0 degrees
- moved R3 199.6 mm to (27.1, 110.0), turned to 0 degrees
- moved TP1 199.2 mm to (363.5, -90.2), turned to 0 degrees
- moved C8 196.3 mm to (38.6, 110.2), turned to 0 degrees
- moved C7 195.3 mm to (39.3, 107.1), turned to 0 degrees
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Connections:
- R10 pad 1: RED_FLASH -> COLON_1
- R11 pad 1: GREEN_FLASH -> COLON_2
- U3 pad 1: DIG_4 -> SEG_E
- U3 pad 10: DIG_6 -> SEG_B
- U3 pad 2: SEG_C -> SEG_D
- U3 pad 3: DIG_5 -> SEG_C
- U3 pad 4: SEG_B -> SEG_DP
- U3 pad 5: SEG_D -> SEG_E
- U3 pad 6: SEG_DP -> SEG_D
- U3 pad 7: SEG_E -> SEG_G
- U3 pad 8: SEG_F -> SEG_C
- U3 pad 9: SEG_G -> SEG_DP
- U5 pad 12: ~{CS0} -> ~{CS}
- U6 pad 17: BZ1_PWM -> unconnected-(U6-IO9-Pad17)
- U6 pad 18: MISO -> unconnected-(U6-IO10-Pad18)
- U6 pad 19: CLK -> unconnected-(U6-IO11-Pad19)
- U6 pad 20: MOSI -> unconnected-(U6-IO12-Pad20)
- U6 pad 21: ~{CS1} -> unconnected-(U6-IO13-Pad21)
- U6 pad 31: LED_EXT1 -> unconnected-(U6-IO38-Pad31)
- U6 pad 32: LED_EXT2 -> unconnected-(U6-IO39-Pad32)
- U6 pad 33: LED_EXT3 -> unconnected-(U6-IO40-Pad33)
- U6 pad 34: MODE -> unconnected-(U6-IO41-Pad34)
- U6 pad 35: RESET -> unconnected-(U6-IO42-Pad35)
- U6 pad 38: SCHRACK_SW -> unconnected-(U6-IO2-Pad38)
- U6 pad 4: ~{CS0} -> unconnected-(U6-IO4-Pad4)
- U6 pad 5: RED_FLASH -> unconnected-(U6-IO5-Pad5)
- U6 pad 6: GREEN_FLASH -> unconnected-(U6-IO6-Pad6)
Routing:
- net SEG_E: track 146.6 -> 0.00 mm, vias 6 -> 0
- net +3V3: track 145.7 -> 0.00 mm, vias 5 -> 0
- net SEG_F: track 143.8 -> 0.00 mm, vias 6 -> 0
- net SEG_A: track 142.6 -> 0.00 mm, vias 6 -> 0
- net SEG_D: track 141.4 -> 0.00 mm, vias 5 -> 0
- net SEG_B: track 129.9 -> 0.00 mm, vias 5 -> 0
- net SEG_DP: track 127.6 -> 0.00 mm, vias 5 -> 0
- net SEG_G: track 125.0 -> 0.00 mm, vias 6 -> 0
- net SEG_C: track 121.3 -> 0.00 mm, vias 5 -> 0
- net MOSI: track 96.9 -> 0.00 mm, vias 4 -> 0
- net DIG_4: track 78.1 -> 0.00 mm, vias 1 -> 0
- net +5V: track 76.6 -> 0.00 mm, vias 3 -> 0
- net DIG_5: track 73.0 -> 0.00 mm, vias 1 -> 0
- net DIG_0: track 70.4 -> 0.00 mm, vias 1 -> 0
- net CLK: track 69.7 -> 0.00 mm, vias 2 -> 0
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- removed copper zone on B.Cu, net GND
- removed copper zone on F.Cu, net GND
Other:
- board text removed: "BOOT"
- board text removed: "D_EXT1"
- board text removed: "D_EXT2"
- board text removed: "D_EXT3"
- board text removed: "EN"
- board text removed: "MADE BY BISMARX"
- board text removed: "PWR_SW"
- board text removed: "SCH_SW"
- board text removed: "SCORE"
- board text removed: "TIME"
- board text removed: "VCC"
- board text removed: "VDD"

Commit message: SchrackMulticlock schematic
Parts:
- removed J2: MEM2067-02-180-00-A_REVB, Schrack_brd:MICRO_SD_CARD
- added C17: 100nF, Capacitor_SMD:C_0805_2012Metric_Pad1.18x1.45mm_HandSolder, F.Cu at (58.8, 100.5)
- added R17: 10k, Resistor_SMD:R_0805_2012Metric_Pad1.20x1.40mm_HandSolder, F.Cu at (55.6, 111.2)
- added R18: 10k, Resistor_SMD:R_0805_2012Metric_Pad1.20x1.40mm_HandSolder, F.Cu at (55.6, 114.2)
- added R19: 10k, Resistor_SMD:R_0805_2012Metric_Pad1.20x1.40mm_HandSolder, F.Cu at (55.6, 117.1)
- added R20: 10k, Resistor_SMD:R_0805_2012Metric_Pad1.20x1.40mm_HandSolder, F.Cu at (55.6, 120.1)
- added R21: 10k, Resistor_SMD:R_0805_2012Metric_Pad1.20x1.40mm_HandSolder, F.Cu at (55.6, 123.0)
- added R22: 10k, Resistor_SMD:R_0805_2012Metric_Pad1.20x1.40mm_HandSolder, F.Cu at (60.3, 111.2)
- added R23: 10k, Resistor_SMD:R_0805_2012Metric_Pad1.20x1.40mm_HandSolder, F.Cu at (60.3, 114.2)
- added R24: 10k, Resistor_SMD:R_0805_2012Metric_Pad1.20x1.40mm_HandSolder, F.Cu at (60.3, 117.1)
- added SW7: SW_Push, Connector_JST:JST_XH_B2B-XH-A_1x02_P2.50mm_Vertical, F.Cu at (42.5, 120.3)
- added SW8: SW_Push, Button_Switch_SMD:SW_SPST_EVQPE1, F.Cu at (65.7, 90.9)
- added SW9: SW_Push, Button_Switch_SMD:SW_SPST_EVQPE1, F.Cu at (65.7, 95.9)
- added U8: 74HC14, Package_SO:SOIC-14_3.9x8.7mm_P1.27mm, F.Cu at (65.4, 83.2)
- added U9: LDD080AUE-101A, Display_7Segment:DA04-11SURKWA, F.Cu at (188.7, 97.4)
- added U9: LDD080AUE-101A, Display_7Segment:DA04-11SURKWA, F.Cu at (167.8, 97.5)
- added U9: LDD080AUE-101A, Display_7Segment:DA04-11SURKWA, F.Cu at (209.4, 97.4)
- C15: value 10uF -> 100nF; footprint Capacitor_Tantalum_SMD:CP_EIA-3216-18_Kemet-A_Pad1.58x1.35mm_HandSolder -> Capacitor_SMD:C_0805_2012Metric_Pad1.18x1.45mm_HandSolder
- R12, R13, R15: value 2k -> 10k
- SW5, SW6: footprint Button_Switch_SMD:SW_SPST_EVQPE1 -> Connector_JST:JST_XH_B2B-XH-A_1x02_P2.50mm_Vertical
- U1: value LM1084-3.3 -> LM1117DT-3.3; footprint Package_TO_SOT_SMD:TO-263-3_TabPin2 -> Package_TO_SOT_SMD:TO-252-3_TabPin2
- moved U4 218.5 mm to (218.3, 76.0)
- moved U3 180.1 mm to (181.6, 76.0)
- moved U2 146.3 mm to (145.1, 76.0)
- moved C7 63.0 mm to (95.9, 79.5)
- moved C8 63.0 mm to (95.3, 82.6)
- moved D4 49.6 mm to (-10.5, 126.4)
- moved R12 36.0 mm to (50.8, 111.2)
- moved R13 36.0 mm to (50.8, 114.2)
- moved R14 36.0 mm to (50.8, 117.1)
- moved R15 36.0 mm to (50.8, 120.1)
- moved R16 36.0 mm to (50.8, 123.0)
- moved C15 25.2 mm to (58.8, 94.5)
- moved U6 24.5 mm to (82.5, 94.6)
- moved SW5 23.9 mm to (42.5, 104.7)
- moved SW6 23.3 mm to (42.5, 112.5)
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Connections:
- C1 pad 1: +5V -> VBATT
- C10 pad 2: MODE -> Net-(C10-Pad2)
- C11 pad 2: SCHRACK_SW -> Net-(C11-Pad2)
- C12 pad 1: EN -> GND
- C12 pad 2: GND -> Net-(C12-Pad2)
- C13 pad 1: GND -> EN
- C13 pad 2: RESET -> GND
- C14 pad 1: BOOT -> GND
- C14 pad 2: GND -> Net-(C14-Pad2)
- C15 pad 1: +3V3 -> GND
- C15 pad 2: GND -> Net-(C15-Pad2)
- C16 pad 1: +3V3 -> GND
- C16 pad 2: GND -> Net-(C16-Pad2)
- C2 pad 1: VBATT -> +5V
- R12 pad 1: MODE -> /MECHANICS/BT1
- R13 pad 1: SCHRACK_SW -> /MECHANICS/BT2
- R14 pad 1: EN -> /MECHANICS/BT2
- R15 pad 1: RESET -> Net-(C10-Pad2)
- R15 pad 2: +3V3 -> /MECHANICS/BT1
- R16 pad 1: ~{CS1} -> Net-(C11-Pad2)
- R16 pad 2: +3V3 -> /MECHANICS/BT2
- SW2 pad 2: MODE -> /MECHANICS/BT1
- SW3 pad 2: SCHRACK_SW -> /MECHANICS/BT2
- SW4 pad 2: RESET -> /MECHANICS/BT2
- SW5 pad 2: EN -> /MECHANICS/MD
- SW6 pad 2: BOOT -> /MECHANICS/BT2
- U5 pad 10: DIG_5 -> unconnected-(U5-DIG_5-Pad10)
- U5 pad 11: DIG_4 -> unconnected-(U5-DIG_1-Pad11)
- U5 pad 2: DIG_0 -> unconnected-(U5-DIG_0-Pad2)
- U5 pad 3: DIG_1 -> unconnected-(U5-DIG_4-Pad3)
- U5 pad 5: DIG_2 -> unconnected-(U5-DIG_6-Pad5)
- U5 pad 6: DIG_3 -> unconnected-(U5-DIG_2-Pad6)
- U5 pad 8: DIG_6 -> unconnected-(U5-DIG_7-Pad8)

Commit message: Schrackcounter Prototype update
Schematic + PCB update, final version
Parts:
- removed BT1: Battery, Battery:BatteryHolder_TruPower_BH-331P_3xAA
- removed BZ1: Buzzer, Schrack_brd:BUZZER_CUI_CPT
- removed C1, C2, C4, C5, C7: 10uF, Capacitor_Tantalum_SMD:CP_EIA-3216-18_Kemet-A_Pad1.58x1.35mm_HandSolder
- removed C10, C11, C12, C13, C14, C15, C16, C17, C3, C6, C8, C9: 100nF, Capacitor_SMD:C_0805_2012Metric_Pad1.18x1.45mm_HandSolder
- removed D1: D_Schottky, Diode_SMD:D_1206_3216Metric_Pad1.42x1.75mm_HandSolder
- removed D2, D3, D5, D6, D7: LED, LED_SMD:LED_0805_2012Metric_Pad1.15x1.40mm_HandSolder
- removed D4: LED, LED_SMD:LED_Cree-PLCC4_3.2x2.8mm_CCW
- removed D_EXT1, D_EXT2, D_EXT3: Conn_01x02_Pin, Connector_JST:JST_XH_B2B-XH-A_1x02_P2.50mm_Vertical
- removed H1, H2, H3, H4: Mounting Hole M3, MountingHole:MountingHole_3.2mm_M3_Pad_Via
- removed J1: TYPE-C-31-M-12 (USB C CONN), sumec_brd:USB_Type_C
- removed R1, R12, R13, R14, R15, R16, R17, R18, R19, R20, R21, R22, R23, R24: 10k, Resistor_SMD:R_0805_2012Metric_Pad1.20x1.40mm_HandSolder
- removed R10, R11, R2, R3, R4, R6, R7: 220R, Resistor_SMD:R_0805_2012Metric_Pad1.20x1.40mm_HandSolder
- removed R5: 0R, Resistor_SMD:R_0805_2012Metric_Pad1.20x1.40mm_HandSolder
- removed R8, R9: 15R, Resistor_SMD:R_0805_2012Metric_Pad1.20x1.40mm_HandSolder
- removed SW1: SW_SPST, Connector_JST:JST_XH_B2B-XH-A_1x02_P2.50mm_Vertical
- removed SW2, SW3, SW4, SW5, SW6, SW7: SW_Push, Connector_JST:JST_XH_B2B-XH-A_1x02_P2.50mm_Vertical
- removed SW8, SW9: SW_Push, Button_Switch_SMD:SW_SPST_EVQPE1
- removed U1: LM1117DT-3.3, Package_TO_SOT_SMD:TO-252-3_TabPin2
- removed U2, U3, U4: LDD080AUE-101A, Schrack_brd:WENRUN_LDD080x_7segment_2dig
- removed U5: MAX7219, Package_SO:SOP-24_7.5x15.4mm_P1.27mm
- removed U6: ESP32-S3-WROOM-2, PCM_Espressif:ESP32-S3-WROOM-2
- removed U7: USBLC6-2SC6, Package_TO_SOT_SMD:TSOT-23-6_HandSoldering
- removed U8: 74HC14, Package_SO:SOIC-14_3.9x8.7mm_P1.27mm
- removed U9 (x3): LDD080AUE-101A, Display_7Segment:DA04-11SURKWA
Other:
- board size 98.5 x 88.5 mm -> 102.6 x 202.3 mm

Commit message: SchrackMulticlock update
Schematic and PCB update
Parts:
- added BT1: Battery, Battery:BatteryHolder_TruPower_BH-331P_3xAA, F.Cu at (-9.46, 64.9)
- added BZ1: Buzzer, Schrack_brd:BUZZER_CUI_CPT, F.Cu at (-48.3, 148.3)
- added C1: 10uF, Capacitor_Tantalum_SMD:CP_EIA-3216-18_Kemet-A_Pad1.58x1.35mm_HandSolder, F.Cu at (2.37, 106.4)
- added C10: 100nF, Capacitor_SMD:C_0805_2012Metric_Pad1.18x1.45mm_HandSolder, F.Cu at (-62.6, 166.9)
- added C10: 100nF, Capacitor_SMD:C_0805_2012Metric_Pad1.18x1.45mm_HandSolder, F.Cu at (248.3, 97.0)
- added C11: 100nF, Capacitor_SMD:C_0805_2012Metric_Pad1.18x1.45mm_HandSolder, F.Cu at (6.98, 117.7)
- added C12: 100nF, Capacitor_SMD:C_0805_2012Metric_Pad1.18x1.45mm_HandSolder, F.Cu at (6.98, 120.8)
- added C13: 100nF, Capacitor_SMD:C_0805_2012Metric_Pad1.18x1.45mm_HandSolder, F.Cu at (6.98, 123.8)
- added C14: 100nF, Capacitor_SMD:C_0805_2012Metric_Pad1.18x1.45mm_HandSolder, F.Cu at (6.98, 126.8)
- added C15: 100nF, Capacitor_SMD:C_0805_2012Metric_Pad1.18x1.45mm_HandSolder, F.Cu at (6.98, 129.8)
- added C16: 100nF, Capacitor_SMD:C_0805_2012Metric_Pad1.18x1.45mm_HandSolder, F.Cu at (6.98, 132.8)
- added C17: 100nF, Capacitor_SMD:C_0805_2012Metric_Pad1.18x1.45mm_HandSolder, F.Cu at (6.98, 135.8)
- added C18: 100nF, Capacitor_SMD:C_0805_2012Metric_Pad1.18x1.45mm_HandSolder, F.Cu at (6.98, 138.8)
- added C2: 10uF, Capacitor_Tantalum_SMD:CP_EIA-3216-18_Kemet-A_Pad1.58x1.35mm_HandSolder, F.Cu at (2.37, 109.5)
- added C3: 100nF, Capacitor_SMD:C_0805_2012Metric_Pad1.18x1.45mm_HandSolder, F.Cu at (17.2, 106.3)
- added C4: 10uF, Capacitor_Tantalum_SMD:CP_EIA-3216-18_Kemet-A_Pad1.58x1.35mm_HandSolder, F.Cu at (2.37, 112.7)
- added C5: 10uF, Capacitor_Tantalum_SMD:CP_EIA-3216-18_Kemet-A_Pad1.58x1.35mm_HandSolder, F.Cu at (-24.6, 73.3)
- added C6: 100nF, Capacitor_SMD:C_0805_2012Metric_Pad1.18x1.45mm_HandSolder, F.Cu at (-19.2, 73.2)
- added C7: 10uF, Capacitor_Tantalum_SMD:CP_EIA-3216-18_Kemet-A_Pad1.58x1.35mm_HandSolder, F.Cu at (44.1, 117.8)
- added C8: 100nF, Capacitor_SMD:C_0805_2012Metric_Pad1.18x1.45mm_HandSolder, F.Cu at (43.5, 120.9)
- added C9: 100nF, Capacitor_SMD:C_0805_2012Metric_Pad1.18x1.45mm_HandSolder, F.Cu at (-62.6, 163.9)
- added C9: 100nF, Capacitor_SMD:C_0805_2012Metric_Pad1.18x1.45mm_HandSolder, B.Cu at (250.4, 102.2)
- added D1: D_Schottky, Diode_SMD:D_1206_3216Metric_Pad1.42x1.75mm_HandSolder, F.Cu at (83.7, 119.5)
- added D1: D_Schottky, Diode_SMD:D_1206_3216Metric_Pad1.42x1.75mm_HandSolder, F.Cu at (247.7, 99.2)
- added D2: LED, LED_SMD:LED_0805_2012Metric_Pad1.15x1.40mm_HandSolder, F.Cu at (-53.2, 159.1)
- added D3: LED, LED_SMD:LED_0805_2012Metric_Pad1.15x1.40mm_HandSolder, F.Cu at (-53.2, 162.1)
- added D4: LED, LED_THT:LED_D5.0mm, F.Cu at (170.9, 72.5)
- added D5: LED, LED_THT:LED_D5.0mm, F.Cu at (170.9, 87.8)
- added D6: LED, LED_THT:LED_D5.0mm, F.Cu at (214.7, 72.5)
- added D7: LED, LED_THT:LED_D5.0mm, F.Cu at (214.7, 87.8)
- added D_EXT1: Conn_01x02_Pin, Connector_JST:JST_XH_B2B-XH-A_1x02_P2.50mm_Vertical, F.Cu at (-61.5, 142.4)
- added D_EXT2: Conn_01x02_Pin, Connector_JST:JST_XH_B2B-XH-A_1x02_P2.50mm_Vertical, F.Cu at (-61.5, 150.2)
- added D_EXT3: Conn_01x02_Pin, Connector_JST:JST_XH_B2B-XH-A_1x02_P2.50mm_Vertical, F.Cu at (-61.5, 158.0)
- added H1: Mounting Hole M3, MountingHole:MountingHole_3.2mm_M3_Pad_Via, F.Cu at (126.6, 63.6)
- added H2: Mounting Hole M3, MountingHole:MountingHole_3.2mm_M3_Pad_Via, F.Cu at (253.6, 63.1)
- added H3: Mounting Hole M3, MountingHole:MountingHole_3.2mm_M3_Pad_Via, F.Cu at (132.1, 119.6)
- added H4: Mounting Hole M3, MountingHole:MountingHole_3.2mm_M3_Pad_Via, F.Cu at (253.6, 119.6)
- added J1: TYPE-C-31-M-12 (USB C CONN), sumec_brd:USB_Type_C, F.Cu at (-44.7, 164.3)
- added J1: TYPE-C-31-M-12 (USB C CONN), sumec_brd:USB_Type_C, F.Cu at (256.3, 100.6)
- added R1: 10k, Resistor_SMD:R_0805_2012Metric_Pad1.20x1.40mm_HandSolder, F.Cu at (-25.3, 76.3)
- added R10: 15R, Resistor_SMD:R_0805_2012Metric_Pad1.20x1.40mm_HandSolder, F.Cu at (248.3, 103.3)
- added R10: 15R, Resistor_SMD:R_0805_2012Metric_Pad1.20x1.40mm_HandSolder, F.Cu at (-33.9, 146.4)
- added R11: 220R, Resistor_SMD:R_0805_2012Metric_Pad1.20x1.40mm_HandSolder, F.Cu at (-33.9, 149.3)
- added R12: 220R, Resistor_SMD:R_0805_2012Metric_Pad1.20x1.40mm_HandSolder, F.Cu at (-33.9, 152.3)
- added R13: 10k, Resistor_SMD:R_0805_2012Metric_Pad1.20x1.40mm_HandSolder, F.Cu at (-1.00, 149.5)
- added R14: 10k, Resistor_SMD:R_0805_2012Metric_Pad1.20x1.40mm_HandSolder, F.Cu at (-1.00, 152.5)
- added R15: 10k, Resistor_SMD:R_0805_2012Metric_Pad1.20x1.40mm_HandSolder, F.Cu at (-1.00, 155.4)
- added R16: 10k, Resistor_SMD:R_0805_2012Metric_Pad1.20x1.40mm_HandSolder, F.Cu at (-1.00, 158.4)
- added R17: 10k, Resistor_SMD:R_0805_2012Metric_Pad1.20x1.40mm_HandSolder, F.Cu at (-1.00, 161.3)
- added R18: 10k, Resistor_SMD:R_0805_2012Metric_Pad1.20x1.40mm_HandSolder, F.Cu at (3.75, 149.5)
- added R19: 10k, Resistor_SMD:R_0805_2012Metric_Pad1.20x1.40mm_HandSolder, F.Cu at (3.75, 152.5)
- added R2: 220R, Resistor_SMD:R_0805_2012Metric_Pad1.20x1.40mm_HandSolder, F.Cu at (-38.6, 140.5)
- added R20: 10k, Resistor_SMD:R_0805_2012Metric_Pad1.20x1.40mm_HandSolder, F.Cu at (3.75, 155.4)
- added R21: 10k, Resistor_SMD:R_0805_2012Metric_Pad1.20x1.40mm_HandSolder, F.Cu at (3.75, 158.4)
- added R22: 10k, Resistor_SMD:R_0805_2012Metric_Pad1.20x1.40mm_HandSolder, F.Cu at (3.75, 161.3)
- added R23: 10k, Resistor_SMD:R_0805_2012Metric_Pad1.20x1.40mm_HandSolder, F.Cu at (8.50, 149.5)
- added R24: 10k, Resistor_SMD:R_0805_2012Metric_Pad1.20x1.40mm_HandSolder, F.Cu at (8.50, 152.5)
- added R25: 10k, Resistor_SMD:R_0805_2012Metric_Pad1.20x1.40mm_HandSolder, F.Cu at (8.50, 155.4)
- added R3: 220R, Resistor_SMD:R_0805_2012Metric_Pad1.20x1.40mm_HandSolder, F.Cu at (-38.6, 143.4)
- added R4: 220R, Resistor_SMD:R_0805_2012Metric_Pad1.20x1.40mm_HandSolder, F.Cu at (-38.6, 146.4)
- added R5: 100k, Resistor_SMD:R_0805_2012Metric_Pad1.20x1.40mm_HandSolder, F.Cu at (-38.6, 149.3)
- added R5: 100k, Resistor_SMD:R_0805_2012Metric_Pad1.20x1.40mm_HandSolder, B.Cu at (252.4, 102.2)
- added R6: 0R, Resistor_SMD:R_0805_2012Metric_Pad1.20x1.40mm_HandSolder, F.Cu at (-38.6, 152.3)
- added R7: 220R, Resistor_SMD:R_0805_2012Metric_Pad1.20x1.40mm_HandSolder, F.Cu at (-38.6, 155.2)
- added R8: 220R, Resistor_SMD:R_0805_2012Metric_Pad1.20x1.40mm_HandSolder, F.Cu at (-33.9, 140.5)
- added R9: 15R, Resistor_SMD:R_0805_2012Metric_Pad1.20x1.40mm_HandSolder, F.Cu at (248.3, 101.3)
- added R9: 15R, Resistor_SMD:R_0805_2012Metric_Pad1.20x1.40mm_HandSolder, F.Cu at (-33.9, 143.4)
- added SW1: SW_SPST, Connector_JST:JST_XH_B2B-XH-A_1x02_P2.50mm_Vertical, F.Cu at (8.85, 108.2)
- added SW2: SW_Push, Connector_JST:JST_XH_B2B-XH-A_1x02_P2.50mm_Vertical, F.Cu at (-9.35, 119.6)
- added SW3: SW_Push, Connector_JST:JST_XH_B2B-XH-A_1x02_P2.50mm_Vertical, F.Cu at (-9.35, 127.4)
- added SW4: SW_Push, Connector_JST:JST_XH_B2B-XH-A_1x02_P2.50mm_Vertical, F.Cu at (-9.35, 135.2)
- added SW5: SW_Push, Connector_JST:JST_XH_B2B-XH-A_1x02_P2.50mm_Vertical, F.Cu at (-9.35, 143.0)
- added SW6: SW_Push, Connector_JST:JST_XH_B2B-XH-A_1x02_P2.50mm_Vertical, F.Cu at (-9.35, 150.8)
- added SW7: SW_Push, Connector_JST:JST_XH_B2B-XH-A_1x02_P2.50mm_Vertical, F.Cu at (-9.35, 158.6)
- added SW8: SW_Push, Button_Switch_SMD:SW_SPST_EVQPE1, F.Cu at (13.9, 129.1)
- added SW9: SW_Push, Button_Switch_SMD:SW_SPST_EVQPE1, F.Cu at (13.9, 134.2)
- added U1: LM1117DT-3.3, Package_TO_SOT_SMD:TO-252-3_TabPin2, F.Cu at (-5.91, 108.8)
- added U2: LDD080AUE-101A, Schrack_brd:WENRUN_LDD080x_7segment_2dig, F.Cu at (131.1, 93.8)
- added U3: LDD080AUE-101A, Schrack_brd:WENRUN_LDD080x_7segment_2dig, F.Cu at (174.9, 93.8)
- added U4: LDD080AUE-101A, Schrack_brd:WENRUN_LDD080x_7segment_2dig, F.Cu at (218.7, 93.8)
- added U5: MAX7219, Package_SO:SOP-24_7.5x15.4mm_P1.27mm, B.Cu at (249.1, 80.5)
- added U6: ESP32-S3-WROOM-2, PCM_Espressif:ESP32-S3-WROOM-2, F.Cu at (208.8, 106.7)
- added U7: USBLC6-2SC6, Package_TO_SOT_SMD:TSOT-23-6_HandSoldering, F.Cu at (-47.3, 170.0)
- added U7: USBLC6-2SC6, Package_TO_SOT_SMD:TSOT-23-6_HandSoldering, B.Cu at (245.8, 102.3)
- added U8: 74HC14, Package_SO:SOIC-14_3.9x8.7mm_P1.27mm, F.Cu at (13.6, 121.5)
- moved TP1 240.1 mm to (178.8, 63.3), turned to 180 degrees
- moved TP2 129.6 mm to (216.6, 64.3), turned to 180 degrees
Routing:
- net /CONNECTIVITY/SHLD: track 0.00 -> 17.5 mm
- net Net-(D1-A): track 0.00 -> 9.84 mm
- net VBUS 5V: track 0.00 -> 6.31 mm, vias 0 -> 1
- net D- IN: track 0.00 -> 6.26 mm
- net D-: track 0.00 -> 4.80 mm
- net D+: track 0.00 -> 4.70 mm
- net GND: track 0.00 -> 4.67 mm
- net D+ IN: track 0.00 -> 4.66 mm
- net Net-(R9-Pad2): vias 0 -> 1
- net Net-(R10-Pad2): vias 0 -> 1
Other:
- board size 102.6 x 202.3 mm -> 270.7 x 88.5 mm
- board text removed: "MODE"
- board text removed: "POWER"
- board text removed: "RESET"

Commit message: SchrackMulticlock update
PCB update
Parts:
- moved TP1 16.8 mm to (178.3, 46.6)
- moved TP2 16.8 mm to (216.1, 47.6)
- moved U6 12.8 mm to (221.6, 108.1)
- moved D4 8.00 mm to (170.9, 64.5)
- moved D5 8.00 mm to (170.9, 79.8)
- moved D6 8.00 mm to (214.7, 64.5)
- moved D7 8.00 mm to (214.7, 79.8)
- moved U2 8.00 mm to (131.1, 85.8)
- moved U3 8.00 mm to (174.9, 85.8)
- moved U4 8.00 mm to (218.7, 85.8)
- moved U5 8.00 mm to (249.1, 72.5)
- moved H2 5.00 mm to (258.6, 63.1)
- moved H1 0.71 mm to (127.1, 63.1)
Other:
- outline, holes or cut-outs redrawn

Commit message: Multiclock pcb update
Parts:
- BT1, U6: moved to B.Cu
- J1: footprint sumec_brd:USB_Type_C -> sumec_brd:HRO_TYPE-C-31-M-12
- moved J1 313.1 mm to (261.1, 97.1), turned to 90 degrees
- moved C10 274.1 mm to (211.0, 151.1)
- moved C9 274.1 mm to (211.0, 148.1)
- moved U7 254.0 mm to (205.6, 146.8), turned to 180 degrees
- moved R5 244.0 mm to (205.3, 154.6)
- moved R9 239.3 mm to (205.3, 150.6)
- moved R10 239.3 mm to (205.3, 152.6)
- moved D1 162.9 mm to (246.6, 125.1)
- moved BT1 153.1 mm to (137.8, 106.9)
- moved BZ1 76.4 mm to (28.1, 148.9)
- moved D2 76.4 mm to (23.2, 159.7)
- moved D3 76.4 mm to (23.2, 162.8)
- moved D_EXT1 76.4 mm to (14.8, 143.0)
- moved D_EXT2 76.4 mm to (14.8, 150.8)
- moved D_EXT3 76.4 mm to (14.8, 158.6)
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Other:
- board size 270.7 x 88.5 mm -> 140 x 59.5 mm

Commit message: SchrackMulticlock and Counter pcb updates
Parts:
- removed the C10 at (285.5, 92.7)
- removed the C9 at (287.7, 98.0)
- removed the D1 at (246.6, 125.1)
- removed the D1 at (284.9, 94.9)
- removed the J1 at (293.6, 96.3)
- removed the R10 at (285.5, 99.0)
- removed the R5 at (289.7, 98.0)
- removed the R9 at (285.5, 97.0)
- removed the U7 at (283.1, 98.1)
- added D1: D_Schottky, Diode_SMD:D_1206_3216Metric_Pad1.42x1.75mm_HandSolder, F.Cu at (248.1, 102.1)
- added D2: D_Schottky, Diode_SMD:D_1206_3216Metric_Pad1.42x1.75mm_HandSolder, F.Cu at (248.1, 99.9)
- added F1: Polyfuse/50R, Fuse:Fuse_0805_2012Metric, F.Cu at (252.5, 100.0)
- added Q1: Q_PMOS, Package_TO_SOT_SMD:SOT-23-3, F.Cu at (248.1, 105.1)
- added R1: 10k, Resistor_SMD:R_0805_2012Metric_Pad1.20x1.40mm_HandSolder, F.Cu at (252.6, 104.0)
- BTss1: renamed from BT1; footprint Battery:BatteryHolder_TruPower_BH-331P_3xAA -> Schrack_brd:SOLDER_PADS; moved to F.Cu
- U7: moved to B.Cu
- moved U1 242.3 mm to (236.3, 103.2), turned to 180 degrees
- moved C2 241.6 mm to (243.8, 100.7), turned to 90 degrees
- moved C4 241.6 mm to (243.8, 105.7), turned to -90 degrees
- moved C1 241.2 mm to (243.5, 111.0), turned to 180 degrees
- moved SW1 240.8 mm to (249.6, 114.3)
- moved R2 231.7 mm to (196.7, 142.9)
- moved C5 231.7 mm to (197.3, 139.8)
- moved C6 231.7 mm to (202.7, 139.8)
- moved C3 226.9 mm to (244.0, 113.1), turned to 180 degrees
- moved BZ1 156.7 mm to (183.8, 166.0)
- moved C11 156.7 mm to (162.7, 134.8)
- moved C12 156.7 mm to (162.7, 137.8)
- moved C13 156.7 mm to (162.7, 140.8)
- moved C14 156.7 mm to (162.7, 143.8)
- moved C15 156.7 mm to (162.7, 146.8)
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- renumbered D2 to D4, D3 to D5, D4 to D6, D5 to D7, D6 to D8, D7 to D9, R9 to R10, R10 to R11, R11 to R12, R12 to R13, R13 to R14, R14 to R15, R15 to R16, R16 to R17, R17 to R18, R18 to R19, R1 to R2, R19 to R20, R20 to R21, R21 to R22, R22 to R23, R23 to R24, R24 to R25, R25 to R26, R2 to R3, R3 to R4, R4 to R5, R5 to R6, R6 to R7, R7 to R8, R8 to R9
Connections:
- SW1 pad 1: +5V -> VBATT
- SW1 pad 2: VBATT -> VBATT_OUT
Routing:
- net VBUS 5V: track 6.31 -> 20.0 mm
- net VBATT_OUT: track 0.00 -> 10.4 mm
- net VBATT: track 0.00 -> 10.2 mm
- net +3V3: track 0.00 -> 9.23 mm
- net +5V: track 0.00 -> 8.00 mm
- net /CONNECTIVITY/SHLD: track 17.5 -> 22.5 mm
- net D-: track 4.80 -> 0.00 mm
- net D+: track 4.70 -> 0.00 mm
- net GND: track 4.67 -> 0.00 mm
- net Net-(D1-A): track 0.00 -> 3.14 mm
- net Net-(R10-Pad2): track 0.00 -> 1.52 mm
- net Net-(R11-Pad2): track 0.00 -> 1.52 mm
- net D+ IN: track 4.66 -> 5.53 mm
Other:
- outline, holes or cut-outs redrawn

Commit message: Multiclock PCB update
Parts:
- BTss1, BZ1, C1, C14, C18, C3, C5, C6, C7, C8, R12, R13, R2, R20, R3, R4, R5, R7, R8, R9: moved to B.Cu
- U6: moved to F.Cu
- moved SW6 119.3 mm to (248.3, 105.8)
- moved J1 106.6 mm to (156.3, 116.8), turned to 0 degrees
- moved SW2 104.5 mm to (248.3, 113.6)
- moved R1 101.1 mm to (151.6, 108.4), turned to -90 degrees
- moved C10 101.0 mm to (151.6, 104.6), turned to 90 degrees
- moved F1 99.4 mm to (153.5, 108.3), turned to -90 degrees
- moved D_EXT3 98.0 mm to (239.3, 105.8)
- moved SW3 97.9 mm to (239.3, 113.6)
- moved R11 97.7 mm to (155.4, 108.3), turned to 90 degrees
- moved R10 96.1 mm to (157.3, 108.3), turned to 90 degrees
- moved R6 94.5 mm to (159.2, 108.3), turned to 90 degrees
- moved D2 94.3 mm to (153.8, 103.9), turned to -90 degrees
- moved C4 93.1 mm to (151.6, 93.4), turned to 90 degrees
- moved C9 92.8 mm to (161.2, 108.3), turned to -90 degrees
- moved R12 92.7 mm to (169.1, 79.1), turned to 90 degrees
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Connections:
- D5 pad 2: VBATT -> VBATT_OUT
- R22 pad 1: /MECHANICS/BT2 -> /MECHANICS/DGT
- R23 pad 1: /MECHANICS/BT2 -> AUX
- R25 pad 2: /MECHANICS/BT2 -> /MECHANICS/DGT
- R26 pad 2: /MECHANICS/BT2 -> AUX
- SW6 pad 2: /MECHANICS/BT2 -> /MECHANICS/DGT
- SW7 pad 2: /MECHANICS/BT2 -> AUX
Routing:
- net /CONNECTIVITY/SHLD: track 22.5 -> 5.53 mm
- net VBUS 5V: track 20.0 -> 4.08 mm
- net +5V: track 8.00 -> 2.53 mm
- net Net-(D1-A): track 3.14 -> 0.00 mm
- net VBATT: track 10.2 -> 7.25 mm
- net VBATT_OUT: track 10.4 -> 12.5 mm
- net Net-(R10-Pad2): track 1.52 -> 0.07 mm
- net Net-(R11-Pad2): track 1.52 -> 0.07 mm
- added copper zone on B.Cu, net GND
- added copper zone on F.Cu, net GND
